File: pcb/typeP/B-ART_typeP.kicad_pcb (KiCad board)
At the start: 2 copper layers, 10.6 x 21.8 mm, 14 parts, among them IC1 BVMCN5103-BK, P1 CONN_01X04, SW1 DIPSW-4

Commit message: pcb: KiCadのプロジェクト名を変更
Parts:
- IC1: footprint uart2ble_bridge:BVMCN5103-BK -> B-ART:BVMCN5103-BK
- SW1: footprint uart2ble_bridge:DIPSW-4P -> B-ART:DIPSW-4P
- W1, W2, W3, W4: footprint uart2ble_bridge:test_th_pad -> B-ART:test_th_pad
Changed lines of the file:
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@@
   (page A4)
   (title_block
-    (title uart2ble_bridge)
+    (title B-ART_typeP)
     (date 2016-11-27)
     (rev 1)
@@
     )
   )
-  (module uart2ble_bridge:BVMCN5103-BK (layer F.Cu)
+  (module B-ART:BVMCN5103-BK (layer F.Cu)
     (at 145.3 110.1)
     (fp_text reference IC1 (at -4.5 -12.25 90) (layer F.SilkS)
@@
       (net 1 +3V3))
   )
-  (module uart2ble_bridge:DIPSW-4P (layer B.Cu)
+  (module B-ART:DIPSW-4P (layer B.Cu)
     (at 146.5 105.5 180)
     (fp_text reference SW1 (at 0.25 0.75 270) (layer B.SilkS)
@@
       (net 2 GND))
   )
-  (module uart2ble_bridge:test_th_pad (layer B.Cu)
+  (module B-ART:test_th_pad (layer B.Cu)
     (at 141.5 101.75)
     (fp_text reference W1 (at 0 -0.5) (layer B.SilkS) hide
@@
       (net 1 +3V3))
   )
-  (module uart2ble_bridge:test_th_pad (layer B.Cu)
+  (module B-ART:test_th_pad (layer B.Cu)
     (at 141.5 104.25)
     (fp_text reference W2 (at 0 -0.5) (layer B.SilkS) hide
@@
       (net 2 GND))
   )
-  (module uart2ble_bridge:test_th_pad (layer B.Cu)
+  (module B-ART:test_th_pad (layer B.Cu)
     (at 141.5 106.75)
     (fp_text reference W3 (at 0 -0.5) (layer B.SilkS) hide
@@
       (net 14 "Net-(IC1-Pad4)"))
   )
-  (module uart2ble_bridge:test_th_pad (layer B.Cu)
+  (module B-ART:test_th_pad (layer B.Cu)
     (at 141.5 109.25)
     (fp_text reference W4 (at 0 -0.5) (layer B.SilkS) hide
