File: pcb/typeU/B-ART_typeU.kicad_pcb (KiCad board)
At the start: 2 copper layers, 12 x 31 mm, 22 parts, among them IC1 FT234XD, IC2 BVMCN5103-BK, P1 USB_A, SW1 DIPSW-4, U1 LXES11D

Commit message: pcb: KiCadのプロジェクト名を変更
Parts:
- IC2: footprint uart2ble_bridge:BVMCN5103-BK -> B-ART:BVMCN5103-BK
- P1: footprint uart2ble_bridge:USB_A_plug -> B-ART:USB_A_plug
- SW1: footprint uart2ble_bridge:DIPSW-4P -> B-ART:DIPSW-4P
- U1: footprint uart2ble_bridge:LXES11D -> B-ART:LXES11D
- W1, W2, W3, W4: footprint uart2ble_bridge:test_th_pad -> B-ART:test_th_pad
Changed lines of the file:
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@@
     )
   )
-  (module uart2ble_bridge:BVMCN5103-BK (layer F.Cu)
+  (module B-ART:BVMCN5103-BK (layer F.Cu)
     (at 168.5 92.25)
     (fp_text reference IC2 (at -4.5 -12.25 90) (layer F.SilkS)
@@
     )
   )
-  (module uart2ble_bridge:DIPSW-4P (layer B.Cu)
+  (module B-ART:DIPSW-4P (layer B.Cu)
     (at 169.75 88.25 180)
     (fp_text reference SW1 (at 0.5 0.25 180) (layer B.SilkS)
@@
       (net 2 GND))
   )
-  (module uart2ble_bridge:LXES11D (layer F.Cu)
+  (module B-ART:LXES11D (layer F.Cu)
     (at 168.25 100.5)
     (fp_text reference U1 (at -1.55 -0.1) (layer F.SilkS)
@@
       (net 2 GND))
   )
-  (module uart2ble_bridge:USB_A_plug (layer F.Cu)
+  (module B-ART:USB_A_plug (layer F.Cu)
     (at 168.5 105.1)
     (fp_text reference P1 (at -4.2 2.1 180) (layer F.SilkS)
@@
       (net 1 "Net-(C1-Pad1)"))
   )
-  (module uart2ble_bridge:test_th_pad (layer B.Cu)
+  (module B-ART:test_th_pad (layer B.Cu)
     (at 164.5 83.5 180)
     (fp_text reference W1 (at 0 -0.5 180) (layer B.SilkS) hide
@@
       (net 4 +3V3))
   )
-  (module uart2ble_bridge:test_th_pad (layer B.Cu)
+  (module B-ART:test_th_pad (layer B.Cu)
     (at 164.5 86)
     (fp_text reference W2 (at 0 -0.5) (layer B.SilkS) hide
@@
       (net 2 GND))
   )
-  (module uart2ble_bridge:test_th_pad (layer B.Cu)
+  (module B-ART:test_th_pad (layer B.Cu)
     (at 164.5 88.5)
     (fp_text reference W3 (at 0 -0.5) (layer B.SilkS) hide
@@
       (net 19 "Net-(IC2-Pad4)"))
   )
-  (module uart2ble_bridge:test_th_pad (layer B.Cu)
+  (module B-ART:test_th_pad (layer B.Cu)
     (at 164.5 91)
     (fp_text reference W4 (at 0 -0.5) (layer B.SilkS) hide
